File: crmx-timo/crmx-timo.kicad_pcb (KiCad board)
At the start: 2 copper layers, 44.5 x 30.5 mm, 27 parts, among them J1 Conn_01x10, J2 Conn_01x08, SW1 SW_Push

Commit message: Logos and description
Routing:
- net GND: vias 16 -> 13
Other:
- board text added: "MHCI CRMX Timo v1.0"
- board text added: "TT"
Changed lines of the file:
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@@
 			(at 0 1.8 0)
 			(layer "B.SilkS")
+			(hide yes)
 			(effects
 				(font
@@
 			(at 0 2.33 90)
 			(layer "B.SilkS")
+			(hide yes)
 			(effects
 				(font
@@
 			(at 0 2.33 90)
 			(layer "B.SilkS")
+			(hide yes)
 			(effects
 				(font
@@
 		)
 	)
+	(gr_poly
+		(pts
+			(xy 212.557999 90.382001) (xy 213.868 90.822) (xy 213.868 90.932) (xy 212.557997 91.372001) (xy 212.557999 91.142)
+			(xy 213.428 90.881999) (xy 212.557999 90.612001)
+		)
+		(stroke
+			(width 0.05)
+			(type solid)
+		)
+		(fill solid)
+		(layer "B.SilkS")
+	)
+	(gr_poly
+		(pts
+			(xy 176.202 100.685999) (xy 175.762001 99.375998) (xy 175.652001 99.375998) (xy 175.212 100.686001)
+			(xy 175.442001 100.685999) (xy 175.702002 99.815998) (xy 175.972 100.685999)
+		)
+		(stroke
+			(width 0.05)
+			(type solid)
+		)
+		(fill solid)
+		(layer "F.SilkS")
+	)
 	(gr_line
 		(start 215.9 77.47)
@@
 		(layer "Edge.Cuts")
 	)
+	(gr_text "TT"
+		(at 213.167998 89.292001 -90)
+		(layer "B.SilkS")
+		(effects
+			(font
+				(face "Inconsolata")
+				(size 1.5 1.5)
+				(thickness 0.3)
+				(bold yes)
+			)
+			(justify mirror)
+		)
+		(render_cache "TT" 270
+			(polygon
+				(pts
+					(xy 212.545498 89.938267) (xy 213.658146 89.938267) (xy 213.658146 90.292907) (xy 213.858547 90.292907)
+					(xy 213.858547 89.336697) (xy 213.658146 89.336697) (xy 213.658146 89.710388) (xy 212.545498 89.710388)
+				)
+			)
+			(polygon
+				(pts
+					(xy 212.545498 88.889) (xy 213.658146 88.889) (xy 213.658146 89.24364) (xy 213.858547 89.24364)
+					(xy 213.858547 88.287429) (xy 213.658146 88.287429) (xy 213.658146 88.661121) (xy 212.545498 88.661121)
+				)
+			)
+		)
+	)
+	(gr_text "MHCI\nCRMX Timo\nv1.0"
+		(at 207.457997 91.582001 270)
+		(layer "B.SilkS")
+		(effects
+			(font
+				(size 1 1)
+				(thickness 0.15)
+			)
+			(justify left bottom mirror)
+		)
+	)
 	(gr_text "SCL"
 		(at 200.66 72.39 0)
@@
 			)
 			(justify right)
+		)
+	)
+	(gr_text "TT"
+		(at 177.292 100.076 0)
+		(layer "F.SilkS")
+		(effects
+			(font
+				(face "Inconsolata")
+				(size 1.5 1.5)
+				(thickness 0.3)
+				(bold yes)
+			)
+		)
+		(render_cache "TT" 0
+			(polygon
+				(pts
+					(xy 176.645733 100.6985) (xy 176.645733 99.585851) (xy 176.291093 99.585851) (xy 176.291093 99.38545)
+					(xy 177.247303 99.38545) (xy 177.247303 99.585851) (xy 176.873612 99.585851) (xy 176.873612 100.6985)
+				)
+			)
+			(polygon
+				(pts
+					(xy 177.695 100.6985) (xy 177.695 99.585851) (xy 177.34036 99.585851) (xy 177.34036 99.38545) (xy 178.296571 99.38545)
+					(xy 178.296571 99.585851) (xy 177.922879 99.585851) (xy 177.922879 100.6985)
+				)
+			)
 		)
 	)
@@
 	)
 	(via
-		(at 210.82 82.55)
-		(size 0.9)
-		(drill 0.4)
-		(layers "F.Cu" "B.Cu")
-		(free yes)
-		(net 7)
-	)
-	(via
-		(at 210.82 88.9)
-		(size 0.9)
-		(drill 0.4)
-		(layers "F.Cu" "B.Cu")
-		(free yes)
-		(net 7)
-	)
-	(via
 		(at 204.47 73.66)
 		(size 0.9)
@@
 		(size 0.9)
 		(drill 0.4)
-		(layers "F.Cu" "B.Cu")
-		(free yes)
-		(net 7)
-	)
-	(via
-		(at 175.26 100.33)
-		(size 0.9)
-		(drill 0.4)
