File: mv-5449/crmx-timo.kicad_pcb (KiCad board)
At the start: 2 copper layers, 32.9 x 30.5 mm, 3 parts, among them J1 Conn_01x10, J2 Conn_01x08

Commit message: Logos and description
Other:
- board text added: "MHCI CTI MV Breakout v1.0"
- board text added: "TT"
Changed lines of the file:
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@@
 		)
+	)
+	(gr_poly
+		(pts
+			(xy 196.361999 91.51) (xy 197.672 91.95) (xy 197.672 92.06) (xy 196.362 92.5) (xy 196.361999 92.27)
+			(xy 197.232 92.01) (xy 196.362 91.74)
+		)
+		(stroke
+			(width 0.05)
+			(type solid)
+		)
+		(fill solid)
+		(layer "B.SilkS")
+	)
+	(gr_poly
+		(pts
+			(xy 211.327999 85.778) (xy 212.637999 85.338) (xy 212.638 85.228) (xy 211.328 84.788) (xy 211.327999 85.018)
+			(xy 212.198 85.278) (xy 211.328 85.548)
+		)
+		(stroke
+			(width 0.05)
+			(type solid)
+		)
+		(fill solid)
+		(layer "F.SilkS")
 	)
 	(gr_line
@@
 		(layer "Edge.Cuts")
 	)
+	(gr_text "TT"
+		(at 196.972 90.42 -90)
+		(layer "B.SilkS")
+		(effects
+			(font
+				(face "Inconsolata")
+				(size 1.5 1.5)
+				(thickness 0.3)
+				(bold yes)
+			)
+			(justify mirror)
+		)
+		(render_cache "TT" 270
+			(polygon
+				(pts
+					(xy 196.3495 91.066266) (xy 197.462148 91.066266) (xy 197.462148 91.420906) (xy 197.662549 91.420906)
+					(xy 197.662549 90.464696) (xy 197.462148 90.464696) (xy 197.462148 90.838387) (xy 196.3495 90.838387)
+				)
+			)
+			(polygon
+				(pts
+					(xy 196.3495 90.016999) (xy 197.462148 90.016999) (xy 197.462148 90.371639) (xy 197.662549 90.371639)
+					(xy 197.662549 89.415428) (xy 197.462148 89.415428) (xy 197.462148 89.78912) (xy 196.3495 89.78912)
+				)
+			)
+		)
+	)
+	(gr_text "MHCI\nCTI MV Breakout\nv1.0"
+		(at 191.262 92.71 -90)
+		(layer "B.SilkS")
+		(effects
+			(font
+				(size 1 1)
+				(thickness 0.15)
+			)
+			(justify left bottom mirror)
+		)
+	)
 	(gr_text "SCL"
 		(at 200.66 72.39 0)
@@
 			)
 			(justify top)
+		)
+	)
+	(gr_text "TT"
+		(at 211.938 86.868 -90)
+		(layer "F.SilkS")
+		(effects
+			(font
+				(face "Inconsolata")
+				(size 1.5 1.5)
+				(thickness 0.3)
+				(bold yes)
+			)
+		)
+		(render_cache "TT" 270
+			(polygon
+				(pts
+					(xy 211.3155 86.221733) (xy 212.428148 86.221733) (xy 212.428148 85.867093) (xy 212.628549 85.867093)
+					(xy 212.628549 86.823303) (xy 212.428148 86.823303) (xy 212.428148 86.449612) (xy 211.3155 86.449612)
+				)
+			)
+			(polygon
+				(pts
+					(xy 211.3155 87.271) (xy 212.428148 87.271) (xy 212.428148 86.91636) (xy 212.628549 86.91636) (xy 212.628549 87.872571)
+					(xy 212.428148 87.872571) (xy 212.428148 87.498879) (xy 211.3155 87.498879)
+				)
+			)
 		)
 	)
@@
 	)
 	(via
-		(at 193.04 81.915)
+		(at 192.024 82.042)
 		(size 0.7)
 		(drill 0.3)
@@
 	)
 	(via
-		(at 195.621673 90.110589)
-		(size 0.7)
-		(drill 0.3)
+		(at 196.85 88.138)
+		(size 0.7)
+		(drill 0.3)
