File: iso-dmx/ISO14xx/iso-dmx.kicad_pcb (KiCad board)
At the start: 2 copper layers, 19 x 23.5 mm, 9 parts, among them J1 Conn_01x06, J2 Conn_01x06, U1 ISO1432BDW, U2 TME-0305S

Commit message: ISO DMX Logos
Routing:
- net GND2: vias 12 -> 9
- net GND1: vias 11 -> 8
Other:
- board text added: "TT"
Changed lines of the file:
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@@
 		)
+	)
+	(gr_poly
+		(pts
+			(xy 84.402 44.038001) (xy 84.841999 42.728) (xy 84.951999 42.728) (xy 85.391999 44.038) (xy 85.161999 44.038001)
+			(xy 84.901999 43.167999) (xy 84.632 44.037999)
+		)
+		(stroke
+			(width 0.05)
+			(type solid)
+		)
+		(fill solid)
+		(layer "B.SilkS")
 	)
 	(gr_line
@@
 			(type dot)
 		)
+		(layer "F.SilkS")
+	)
+	(gr_poly
+		(pts
+			(xy 91.796001 45.976) (xy 90.486 46.416) (xy 90.486 46.526) (xy 91.796 46.966) (xy 91.796001 46.736)
+			(xy 90.926 46.476) (xy 91.796 46.206)
+		)
+		(stroke
+			(width 0.05)
+			(type solid)
+		)
+		(fill solid)
 		(layer "F.SilkS")
 	)
@@
 		(layer "Edge.Cuts")
 	)
+	(gr_text "TT"
+		(at 83.312 43.428 0)
+		(layer "B.SilkS")
+		(effects
+			(font
+				(face "Inconsolata")
+				(size 1.5 1.5)
+				(thickness 0.3)
+				(bold yes)
+			)
+			(justify mirror)
+		)
+		(render_cache "TT" 0
+			(polygon
+				(pts
+					(xy 83.958266 44.0505) (xy 83.958266 42.937851) (xy 84.312906 42.937851) (xy 84.312906 42.73745)
+					(xy 83.356696 42.73745) (xy 83.356696 42.937851) (xy 83.730387 42.937851) (xy 83.730387 44.0505)
+				)
+			)
+			(polygon
+				(pts
+					(xy 82.908999 44.0505) (xy 82.908999 42.937851) (xy 83.263639 42.937851) (xy 83.263639 42.73745)
+					(xy 82.307428 42.73745) (xy 82.307428 42.937851) (xy 82.68112 42.937851) (xy 82.68112 44.0505)
+				)
+			)
+		)
+	)
 	(gr_text "DE"
 		(at 81.788 59.055 0)
@@
 		)
 	)
+	(gr_text "TT"
+		(at 91.186 44.886 90)
+		(layer "F.SilkS")
+		(effects
+			(font
+				(face "Inconsolata")
+				(size 1.5 1.5)
+				(thickness 0.3)
+				(bold yes)
+			)
+		)
+		(render_cache "TT" 90
+			(polygon
+				(pts
+					(xy 91.8085 45.532266) (xy 90.695851 45.532266) (xy 90.695851 45.886906) (xy 90.49545 45.886906)
+					(xy 90.49545 44.930696) (xy 90.695851 44.930696) (xy 90.695851 45.304387) (xy 91.8085 45.304387)
+				)
+			)
+			(polygon
+				(pts
+					(xy 91.8085 44.482999) (xy 90.695851 44.482999) (xy 90.695851 44.837639) (xy 90.49545 44.837639)
+					(xy 90.49545 43.881428) (xy 90.695851 43.881428) (xy 90.695851 44.25512) (xy 91.8085 44.25512)
+				)
+			)
+		)
+	)
 	(gr_text "ISO143x"
 		(at 83.82 50.292 0)
@@
 	)
 	(via
-		(at 92.075 44.577)
-		(size 0.7)
-		(drill 0.3)
-		(layers "F.Cu" "B.Cu")
-		(free yes)
-		(net 2)
-	)
-	(via
 		(at 85.725 59.9694)
 		(size 0.7)
@@
 	(via
 		(at 85.725 56.1594)
-		(size 0.7)
-		(drill 0.3)
-		(layers "F.Cu" "B.Cu")
-		(free yes)
-		(net 2)
-	)
-	(via
-		(at 92.075 45.974)
-		(size 0.7)
-		(drill 0.3)
-		(layers "F.Cu" "B.Cu")
-		(free yes)
-		(net 2)
-	)
-	(via
-		(at 92.075 47.371)
 		(size 0.7)
 		(drill 0.3)
@@
 		(size 0.7)
 		(drill 0.3)
-		(layers "F.Cu" "B.Cu")
-		(free yes)
-		(net 4)
-	)
-	(via
-		(at 75.565 47.371)
-		(size 0.7)
-		(drill 0.3)
-		(layers "F.Cu" "B.Cu")
-		(free yes)
-		(net 4)
-	)
-	(via
-		(at 75.565 44.577)
-		(size 0.7)
-		(drill 0.3)
-		(layers "F.Cu" "B.Cu")
-		(free yes)
-		(net 4)
-	)
-	(via
-		(at 75.565 45.974)
-		(size 0.7)
-		(drill 0.3)
