File: a6211/a6211.kicad_pcb (KiCad board)
At the start: 2 copper layers, 60 x 25 mm, 26 parts, among them J1 Conn_01x02, J2 Conn_01x02, J3 Conn_01x07, J4 Conn_01x05, J5 Conn_01x02, U1 A6211

Commit message: A6211 Production v1
Parts:
- added HS1: Heatsink, MHCI:HSB02-101007, B.Cu at (149.8, 131.0)
- J3, J4, J5: moved to B.Cu
- R2, R3, R4, R5: footprint Resistor_SMD:R_0612_1632Metric_Pad1.18x3.40mm_HandSolder -> Resistor_SMD:R_1206_3216Metric
- turned J3 to -90 degrees
- turned J4 to 90 degrees
- turned J5 to 0 degrees
Routing:
- net EN: track 37.7 -> 60.4 mm, vias 1 -> 0
- net GND: track 0.00 -> 1.39 mm, vias 37 -> 73
- net Net-(JP4-A): track 1.91 -> 1.29 mm
- net Net-(JP3-A): track 1.91 -> 1.29 mm
- net Net-(JP2-A): track 1.91 -> 1.29 mm
- net Net-(JP1-A): track 1.91 -> 1.29 mm
- net LED-: vias 22 -> 31
- net /SW: vias 11 -> 38
Other:
- board text added: "0.9A"
- board text added: "1.3A"
- board text added: "2.4A"
- board text added: "2.7A"
- board text added: "EN"
- board text added: "GND"
- board text added: "Input: 6-48V Output: 2.7A Max"
- board text added: "LED+"
- board text added: "LED-"
- board text added: "Lighting Systems A6211 Driver v1.0"
- board text added: "NC"
- board text added: "VCC"
