File: a6211/a6211.kicad_pcb (KiCad board)
At the start: 2 copper layers, 60 x 25 mm, 27 parts, among them J1 Conn_01x02, J2 Conn_01x02, J3 Conn_01x07, J4 Conn_01x05, J5 Conn_01x02, U1 A6211

Commit message: Walkure motherboard production v1.0
Other:
- board text added: "Flip these around so ground runs back into the chip See eval board"
Changed lines of the file:
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@@
+		)
+	)
+	(gr_text "Flip these around so ground\nruns back into the chip\nSee eval board"
+		(at 165.56 138.85 0)
+		(layer "Dwgs.User")
+		(effects
+			(font
+				(size 0.66 0.66)
+				(thickness 0.1)
+			)
 		)
 	)
@@
 		(start 190.399999 115.399999)
 		(end 192 117)
+		(width 1.6)
+		(layer "F.Cu")
+		(net 7)
+	)
+	(segment
+		(start 185.42 135.89)
+		(end 187.96 135.89)
 		(width 1.6)
 		(layer "F.Cu")
@@
 		(width 1.6)
 		(layer "B.Cu")
-		(net 7)
-	)
-	(segment
-		(start 187.96 135.89)
-		(end 185.42 135.89)
-		(width 1.6)
-		(layer "B.Cu")

Commit message: A6211 BOM files
Parts:
- D1: value D_Schottky -> Diode
- L1: value L -> Inductor
- R1: value R_US -> 120k
Changed lines of the file:
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@@
 			)
 		)
-		(property "Value" "L"
+		(property "Value" "Inductor"
 			(at 0 6.35 0)
 			(layer "F.Fab")
@@
 			)
 		)
-		(property "Value" "D_Schottky"
+		(property "Value" "Diode"
 			(at 0 4.2 0)
 			(layer "F.Fab")
@@
 			)
 		)
-		(property "Value" "R_US"
+		(property "Value" "120k"
 			(at 0 1.43 0)
 			(layer "F.Fab")

Commit message: Make GND connections use spokes to reduce soldering issues
Other:
- board text added: "Lighting Systems A6211 Driver v1.1"
- board text removed: "Lighting Systems A6211 Driver v1.0"
Changed lines of the file:
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@@
 		)
 	)
-	(gr_text "Lighting\nSystems\nA6211 Driver\nv1.0"
+	(gr_text "Lighting\nSystems\nA6211 Driver\nv1.1"
 		(at 176.42 131.85 0)
 		(layer "F.SilkS")
@@
 			)
 		)
+	)
+	(zone
+		(net 2)
+		(net_name "GND")
+		(layers "F&B.Cu")
+		(hatch edge 0.5)
+		(priority 8)
+		(connect_pads
+			(clearance 0.5)
+		)
+		(min_thickness 0.25)
+		(filled_areas_thickness no)
+		(fill yes
+			(thermal_gap 0.5)
+			(thermal_bridge_width 0.5)
+		)
+		(polygon
+			(pts
+				(xy 148 113.8) (xy 148 117.6) (xy 156.3 117.6) (xy 156.3 113.7)
+			)
+		)

Commit message: A6211 v1.1
Parts:
- removed JP2, JP3, JP4: ~, Jumper:SolderJumper-2_P1.3mm_Open_RoundedPad1.0x1.5mm
- removed R1: 120k, Resistor_SMD:R_0603_1608Metric_Pad0.98x0.95mm_HandSolder
- removed R4: 0.082R, Resistor_SMD:R_1206_3216Metric
- removed R5: 0.075R, Resistor_SMD:R_1206_3216Metric
- added C8: 470nF, Capacitor_SMD:C_1206_3216Metric, F.Cu at (170.8, 127.4)
- C3: value 100nF -> 47nF
- C7: value Cout -> 2.2uF; footprint Capacitor_SMD:C_0603_1608Metric_Pad1.08x0.95mm_HandSolder -> Capacitor_SMD:C_1206_3216Metric
- D1: value Diode -> D_Schottky
- JP1: value ~ -> Jumper_3_Open; footprint Jumper:SolderJumper-2_P1.3mm_Open_RoundedPad1.0x1.5mm -> Jumper:SolderJumper-3_P1.3mm_Open_RoundedPad1.0x1.5mm_NumberLabels
- L1: value Inductor -> 10uH; footprint Inductor_SMD:L_10.4x10.4_H4.8 -> Inductor_SMD:L_Coilcraft_XAL6060-XXX
- R2: value 0.22R -> 120k; footprint Resistor_SMD:R_1206_3216Metric -> Resistor_SMD:R_0603_1608Metric_Pad0.98x0.95mm_HandSolder
- moved JP1 12.7 mm to (172.1, 131.0), turned to 0 degrees
- moved R2 11.4 mm to (151.8, 126.8), turned to 0 degrees
- moved R3 4.00 mm to (162.8, 131.2), turned to 180 degrees
- moved C6 3.35 mm to (153.0, 131.5), turned to -90 degrees
- moved L1 1.90 mm to (166.8, 120.7)
- moved C5 1.55 mm to (154.5, 131.5), turned to -90 degrees
- moved C7 0.72 mm to (173.2, 127.4)
Connections:
- C7 pad 2: LED- -> Net-(JP1-B)
- R2 pad 1: Net-(JP1-A) -> VCC
- R2 pad 2: GND -> Net-(U1-TON)
- R3 pad 1: Net-(JP2-A) -> LED-
Routing:
- net LED-: track 6.89 -> 25.8 mm, vias 31 -> 0
- net Net-(JP1-B): track 0.00 -> 2.21 mm
- net GND: track 1.39 -> 0.00 mm, vias 73 -> 87
- net Net-(JP4-A): track 1.29 -> 0.00 mm
- net Net-(JP3-A): track 1.29 -> 0.00 mm
- net Net-(JP2-A): track 1.29 -> 0.00 mm
- net Net-(JP1-A): track 1.29 -> 2.14 mm
- net EN: track 60.4 -> 61.0 mm
- net LED+: vias 10 -> 17
- net /SW: vias 38 -> 28
- removed copper zone on B.Cu, net LED-
Other:
- board text added: "Vin: 42V Iled: 1.3A Fsw: 600kHz"
- board text removed: "0.9A"
- board text removed: "2.4A"
- board text removed: "2.7A"
- board text removed: "Flip these around so ground runs back into the chip See eval board"
- board text removed: "Input: 6-48V Output: 2.7A Max"

Commit message: A6211 - cheaper inductor
Parts:
- removed L1: 10uH, Inductor_SMD:L_Coilcraft_XAL6060-XXX
- added L2: 10uH, Inductor_SMD:L_10.4x10.4_H4.8, F.Cu at (168.5, 119.5)
- C8: footprint Capacitor_SMD:C_1206_3216Metric -> Capacitor_SMD:C_0805_2012Metric
- moved C8 0.60 mm to (170.8, 128.0)
Routing:
- net LED-: track 25.8 -> 28.0 mm
- net EN: track 61.0 -> 59.7 mm
- net LED+: vias 17 -> 16
- net GND: vias 87 -> 86
- net /SW: vias 28 -> 21

Commit message: A6211 v1.1
Parts:
- removed C7: 2.2uF, Capacitor_SMD:C_1206_3216Metric
- removed C8: 470nF, Capacitor_SMD:C_0805_2012Metric
- removed JP1: Jumper_3_Open, Jumper:SolderJumper-3_P1.3mm_Open_RoundedPad1.0x1.5mm_NumberLabels
- C3: value 47nF -> 100nF
Routing:
- net Net-(JP1-B): track 2.21 -> 0.00 mm
- net Net-(JP1-A): track 2.06 -> 0.00 mm
- net LED-: track 28.0 -> 26.7 mm
- net GND: vias 86 -> 94
Other:
- board text added: "Lighting Systems A6211 Driver v1.2"
- board text removed: "Lighting Systems A6211 Driver v1.1"
