File: walkure-motherboard/Driver.kicad_sch (KiCad schematic)
At the start: 2 parts, among them J2 Conn_01x02

Commit message: Walkure motherboard v1.0 schematic
Connections:
- net LED+: now also J2.1 (Pin_1); no longer J2.2 (Pin_2)
- net LED-: now also J2.2 (Pin_2); no longer J2.1 (Pin_1)
Changed lines of the file:
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@@
 	(paper "A4")
-	(label "LED-"
-		(at 165.1 86.36 180)
-		(fields_autoplaced yes)
-		(effects
-			(font
-				(size 1.27 1.27)
-			)
-			(justify right bottom)
-		)
-	)
 	(label "LED-"
 		(at 148.59 90.17 0)
@@
 		)
 	)
-	(label "LED+"
+	(label "LED-"
 		(at 165.1 88.9 180)
 		(fields_autoplaced yes)
@@
 		)
 	)
+	(label "LED+"
+		(at 165.1 86.36 180)
+		(fields_autoplaced yes)
+		(effects
+			(font
+				(size 1.27 1.27)
+			)
+			(justify right bottom)
+		)
+	)

Commit message: Walkure motherboard production v1.0
Parts:
- renumbered J2 to J4, U1 to U5
Changed lines of the file:
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@@
 		(dnp no)
 		(fields_autoplaced yes)
-		(property "Reference" "J2"
+		(property "Reference" "J4"
 			(at 172.72 86.3599 0)
 			(effects
@@
 		(dnp no)
 		(fields_autoplaced yes)
-		(property "Reference" "U1"
+		(property "Reference" "U5"
 			(at 138.43 77.47 0)
 			(effects
