File: walkure-motherboard/walkure-motherboard.kicad_sch (KiCad schematic)
At the start: 4 parts, among them J7 Conn_01x02, J8 Conn_01x02, J9 Conn_01x02

Commit message: Walkure motherboard v1.0 schematic
Parts:
- added J10: Conn_01x02, MHCI:2060-452-998-404 Wago, symbol Connector_Generic:Conn_01x02
- added J11, J20, J21, J22: Conn_01x03, Connector_PinHeader_2.54mm:PinHeader_1x03_P2.54mm_Vertical, symbol Connector_Generic:Conn_01x03
- added J12, J13, J14, J15, J16, J17, J18, J19: Conn_01x04, Connector_PinHeader_2.54mm:PinHeader_1x04_P2.54mm_Vertical, symbol Connector_Generic:Conn_01x04
- added JP1, JP2, JP3, JP4: SolderJumper_2_Open, Jumper:SolderJumper-2_P1.3mm_Open_RoundedPad1.0x1.5mm, symbol Jumper:SolderJumper_2_Open
- added U10: DS18B20Z, Package_SO:SOIC-8_3.9x4.9mm_P1.27mm, symbol Sensor_Temperature:DS18B20Z
- added U11: 74LS04, Package_DIP:DIP-14_W7.62mm_Socket, symbol 74xx:74LS04
- added U12: TSR_2-2450, Converter_DCDC:Converter_DCDC_TRACO_TSR-1_THT, symbol Regulator_Switching:TSR_1-2450
- added U8: ~, MHCI:ESP-32-S3-Zero - PTH, symbol MHCI:ESP32-S3-Zero
- added U9: LTV-827, Package_DIP:DIP-8_W7.62mm_Socket, symbol Isolator:LTV-827
Connections:
- net GND: now also J10.2 (Pin_2), J11.3 (Pin_3), J12.1 (Pin_1), J13.1 (Pin_1), J14.1 (Pin_1), J15.1 (Pin_1), J16.1 (Pin_1), J17.1 (Pin_1), J18.1 (Pin_1), J19.1 (Pin_1), J20.3 (Pin_3), J21.3 (Pin_3), J22.3 (Pin_3), U10.5 (GND), U12.2 (GND), U8.GND
- net +5V: now reaches U2.1 (VIN)
- net +5V: now also U2.3 (5V), U2.4 (5V), U2.5 (5V), U2.6 (5V), U12.3 (Vout), U8.5V
- net SDA: now reaches U2.17 (SDA)
- net SDA: now also JP1.1 (A)
- net SCL: now reaches U2.18 (SCL)
- net SCL: now also JP2.1 (A)
- net RX: now reaches U2.19 (RX)
- net RX: now also JP3.2 (B)
- net TX: now reaches U2.20 (TX)
- net TX: now also JP4.2 (B)
- new net: JP2.2 (B), U8.2 (GPIO2)
- new net: JP1.2 (B), U8.1 (GPIO1)
- new net: JP3.1 (A), U8.TX
- new net: JP4.1 (A), U8.RX
- new net +12V: J10.1 (Pin_1), J12.2 (Pin_2), J13.2 (Pin_2), J14.2 (Pin_2), J15.2 (Pin_2), J16.2 (Pin_2), J17.2 (Pin_2), J18.2 (Pin_2), J19.2 (Pin_2), U12.1 (Vin)
- new net +3V3: J11.1 (Pin_1), J20.1 (Pin_1), J21.1 (Pin_1), J22.1 (Pin_1), U10.3 (V_{DD}), U8.3V3
- new net FAN1: J12.4 (Pin_4), J13.4 (Pin_4), J14.4 (Pin_4), J15.4 (Pin_4)
- new net FAN2: J18.4 (Pin_4), J19.4 (Pin_4)
- new net FAN3: J16.4 (Pin_4), J17.4 (Pin_4)
- new net TEMP1: J11.2 (Pin_2), J20.2 (Pin_2)
- new net TEMP2: J21.2 (Pin_2), J22.2 (Pin_2)
- new net TEMP3: U10.4 (DQ)
- no-connect marks 0 -> 10
Other:
- note added: "CURRENT LIMIT RESISTORS - option 5V PSU Fan controller board 12V power input Silkscreen and labelling LEDs Gaps for SDA, SCL, and TX, RX"
- note removed: "CURRENT LIMIT RESISTORS 5V PSU Fan controller board 12V power input Silkscreen and labelling"
- moved on the sheet: J7, J8, J9, U2

Commit message: Adding fans and breakouts
Parts:
- removed U11: 74LS04, Package_DIP:DIP-14_W7.62mm_Socket, symbol 74xx:74LS04
- removed U9: LTV-827, Package_DIP:DIP-8_W7.62mm_Socket, symbol Isolator:LTV-827
- added JP5: SolderJumper_3_Open, Jumper:SolderJumper-3_P1.3mm_Open_RoundedPad1.0x1.5mm, symbol Jumper:SolderJumper_3_Open
- added JP6, JP7: SolderJumper_2_Open, Jumper:SolderJumper-2_P1.3mm_Open_RoundedPad1.0x1.5mm, symbol Jumper:SolderJumper_2_Open
- added U13: TXB0102DCU, Package_SO:VSSOP-8_2.3x2mm_P0.5mm, symbol Logic_LevelTranslator:TXB0102DCU
Connections:
- net +3V3: now also JP5.1 (A), U13.3 (VCCA), U13.6 (OE)
- net +5V: now also JP5.3 (B)
- net GND: now also U13.2 (GND)
- net SCL: now also JP7.1 (A), U13.4 (A2); no longer U2.18 (SCL)
- net SDA: now also JP6.1 (A), U13.5 (A1); no longer U2.17 (SDA)
- new net: JP5.2 (C), U13.7 (VCCB)
- new net SCL_5: JP7.2 (B), U13.1 (B2), U2.18 (SCL)
- new net SDA_5: JP6.2 (B), U13.8 (B1), U2.17 (SDA)
Other:
- note added: "5V PSU Fan controller board 12V power input Silkscreen and labelling Optically isoalted fan LEDs"
- note removed: "CURRENT LIMIT RESISTORS - option 5V PSU Fan controller board 12V power input Silkscreen and labelling LEDs Gaps for SDA, SCL, and TX, RX"
- moved on the sheet: J10, J11, J12, J13, J14, J15, J16, J17, J18, J19, J20, J21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

Commit message: Walkure motherboard production v1.0
Parts:
- removed U12: TSR_2-2450, Converter_DCDC:Converter_DCDC_TRACO_TSR-1_THT, symbol Regulator_Switching:TSR_1-2450
- added D1, D2, D3: D_Schottky, Diode_THT:D_DO-41_SOD81_P5.08mm_Vertical_AnodeUp, symbol Device:D_Schottky
- added F1: Fuse, MHCI:Keystone 4628, symbol Device:Fuse
- added H1, H2, H3, H4, H5, H6: MountingHole, MountingHole:MountingHole_3.2mm_M3_ISO14580, symbol Mechanical:MountingHole
- added JP8, JP9: SolderJumper_2_Open, Jumper:SolderJumper-2_P1.3mm_Open_RoundedPad1.0x1.5mm, symbol Jumper:SolderJumper_2_Open
- added TP1, TP14, TP15, TP16, TP17, TP18, TP19, TP2, TP24, TP25, TP26, TP27, TP3, TP4, TP5, TP6, TP7: TestPoint, TestPoint:TestPoint_Pad_D2.0mm, symbol Connector:TestPoint
Connections:
- net +12V: now also U2.1 (VIN), F1.1, TP1.1; no longer J10.1 (Pin_1)
- net +3V3: now also JP9.2 (B), TP3.1
- net +5V: now also U2.24 (5V), JP8.2 (B), TP2.1; no longer U2.1 (VIN), U2.6 (5V), U8.5V
- net FAN1: now also U8.4 (GPIO4), D1.1 (K), TP14.1
- net FAN2: now also U8.5 (GPIO5), D2.1 (K), TP15.1
- net FAN3: now also U8.6 (GPIO6), D3.1 (K), TP16.1
- net GND: now also U2.2 (GND_IN), U2.23 (GND), U2.26 (GND), D1.2 (A), D2.2 (A), D3.2 (A), TP26.1, TP27.1, TP4.1
- net RX: now also TP24.1
- net TEMP1: now also U8.7 (GPIO7), TP17.1
- net TEMP2: now also U8.8 (GPIO8), TP18.1
- net TEMP3: now also U8.9 (GPIO9), TP19.1
- net TX: now also TP25.1
- net VCC 1: now also TP5.1
- net VCC 2: now also TP6.1
- net VCC 3: now also TP7.1
- new net: F1.2, J10.1 (Pin_1)
- new net: JP9.1 (A), U2.25 (3V3)
- new net: JP8.1 (A), U8.5V
- no-connect marks 10 -> 16
Other:
- note removed: "5V PSU Fan controller board 12V power input Silkscreen and labelling Optically isoalted fan LEDs"
- moved on the sheet: J10, J7, J8, J9, JP1, JP2, JP3, JP4, JP5, JP6, JP7, U13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
