File: tps922055/tps922055/tps922055.kicad_sch (KiCad schematic)
At the start: 29 parts, among them J1 Conn_01x02, J2 Conn_01x05, J3 Conn_01x07, J4 Conn_01x02, U1 TPS922052DRRR

Commit message: Cheaper diode
Parts:
- D1: LCSC C145187 -> C151733; LCSC_Alt (none) -> C145187
Changed lines of the file:
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@@
 			)
 		)
-		(property "LCSC" "C145187"
+		(property "LCSC" "C151733"
 			(at 148.59 49.53 90)
 			(effects
+				(font
+					(size 1.27 1.27)
+				)
+				(hide yes)
+			)
+		)
+		(property "LCSC_Alt" "C145187"
+			(at 148.59 49.53 90)
+			(effects

Commit message: Schematic needs vias
Parts:
- removed JP3: Jumper_2_Open, Jumper:SolderJumper-2_P1.3mm_Open_RoundedPad1.0x1.5mm, symbol Jumper:Jumper_2_Open
Connections:
- net FAULT is gone; now on net GND: U1.5 (FAULT)
- net VCC: no longer C3.1, C4.1, C6.1, C7.1, D1.1 (K), J1.2 (Pin_2), J2.1 (Pin_1), J2.2 (Pin_2), J3.1 (Pin_1), J3.2 (Pin_2), J4.1 (Pin_1), R9.1, U1.1 (VIN)
- new net VDD: C3.1, C4.1, C6.1, C7.1, D1.1 (K), J1.2 (Pin_2), J2.1 (Pin_1), J2.2 (Pin_2), J3.1 (Pin_1), J3.2 (Pin_2), J4.1 (Pin_1), R9.1, U1.1 (VIN)

Commit message: TPS Layout complete
Parts:
- added D2: D_Schottky, Diode_SMD:D_SMC, symbol Device:D_Schottky
- added JP5: Jumper_3_Open, Jumper:SolderJumper-3_P1.3mm_Open_RoundedPad1.0x1.5mm, symbol Jumper:Jumper_3_Open
- added L2: 10uH, Inductor_SMD:L_Coilcraft_XAL6060-XXX, symbol Device:L
- added R10: 56k, Resistor_SMD:R_0603_1608Metric, symbol Device:R_US
- C4: LCSC C28233 -> C14663
- C7: value 0.1uF -> 100nF; LCSC C28233 -> C14663
- D1: now not fitted; now left out of the parts list
- L1: LCSC C5329540 -> C19191628
- R1: value R_US -> 56k
- R2: value R_US -> 27k
Connections:
- net FSET: now also R10.1
- net GND: now also JP5.2 (C); no longer R2.2
- net SW: now also D2.2 (A); no longer D1.2 (A)
- net VDD: now also D2.1 (K); no longer D1.1 (K)
- new net: JP5.1 (A), R2.2
- new net: JP5.3 (B), R10.2
Other:
- note added: "Ccomp: 10nF (x2) on eval board. 1nF (x1) from datasheet 0.01uF 10V 0603"
- note added: "Ccout: 0.1uF + 1uF 100V 0603, 0805"
- note added: "Cflt: 2.2uF (eval) 1nF (datasheet) 16V 0603"
- note added: "Cvcc: 1uF 25V 0603"
- note added: "Cvin: 100nF 100V 0603"
- note added: "Rflt: 825R (eval), 100R (datasheet) 0.1% 0.1W 0603"
- note added: "Rfset: 27k 0.1% 0.1W 0603 -> 800kHz Rfset2: 56k 0.1% 0.1W 0603 -> 400kHz"
- note added: "Rtemp: 56k 0.1% 0.1W 0603 -> 110degC"
- note removed: "Ccomp 10nF (x2) on eval board. 1nF (x1) from datasheet 0.01uF 10V 0603"
- note removed: "Ccout 0.1uF (x1) 1uF (x1) 100V 0603, 0805"
- note removed: "Cflt 2.2uF (eval) 1nF (datasheet) 16V 0603"
- note removed: "Cvcc 1uF (eval) (datasheet) 25V 0603"
- note removed: "Cvin 100nF (eval) (datasheet) 100V 0603"
- note removed: "Rflt 825R (eval), 100R (datasheet) 0.1% 0.1W 0603"
- note removed: "Rfset 102k = 250kHz 0.1% 0.1W 0603 27k = 800kHz"
- note removed: "Rtemp 100 deg = ~60k (lower val = higher temp 0.1% 0.1W 0603 56k = ~110"
- moved on the sheet: C1, C2, C3, C4, C5, C6, C7, H1, H2, HS1, J1, J2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

Commit message: TPS922052 - Larger inductor
Parts:
- removed C6: 15uF, Capacitor_SMD:CP_Elec_10x10.5, symbol Device:C_Polarized_US
- added C8: 47uF, Capacitor_SMD:CP_Elec_8x10, symbol Device:C_Polarized_Small_US
- added C9: 4.7uF, Capacitor_SMD:C_1206_3216Metric, symbol Device:C_Small
- added L3: 15uH, Inductor_SMD:L_Coilcraft_XAL6060-XXX, symbol Device:L
- L1: value 10uH -> 22uH; footprint Inductor_SMD:L_Coilcraft_XAL6060-XXX -> Inductor_SMD:L_10.4x10.4_H4.8; LCSC C19191628 -> C10165
Connections:
- net GND: now also C8.2, C9.2
- net VDD: now also C8.1, C9.1

Commit message: Update Tset value to 120 degC
Parts:
- R1: value 56k -> 27k; LCSC C23206 -> C22967
Other:
- note added: "Rtemp: 27k 0.1% 0.1W 0603 -> 120degC"
- note removed: "Rtemp: 56k 0.1% 0.1W 0603 -> 110degC"
Changed lines of the file:
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@@
 		)
 	)
-	(text "Rtemp: 56k 0.1% 0.1W 0603 -> 110degC\n"
+	(text "Rtemp: 27k 0.1% 0.1W 0603 -> 120degC\n"
 		(exclude_from_sim no)
 		(at 144.526 126.238 0)
@@
 			)
 		)
-		(property "Value" "56k"
+		(property "Value" "27k"
 			(at 153.67 93.9799 0)
 			(effects
@@
 			)
 		)
-		(property "LCSC" "C23206"
+		(property "LCSC" "C22967"
 			(at 151.13 92.71 0)
 			(effects

Commit message: TPS922052 v1.0
Parts:
- added JP3: Jumper_2_Open, Jumper:SolderJumper-2_P1.3mm_Open_RoundedPad1.0x1.5mm, symbol Jumper:Jumper_2_Open
Connections:
- net LED-: now also JP3.1 (A); no longer C3.2, C7.2
- new net OUTCAP: C3.2, C7.2, JP3.2 (B)
Other:
- note added: "Ccomp: 1nF 0.01uF 10V 0603"
- note added: "Cflt: 1nF 16V 0603"
- note added: "Rflt: 100R 0.1% 0.1W 0603"
- note removed: "Ccomp: 10nF (x2) on eval board. 1nF (x1) from datasheet 0.01uF 10V 0603"
- note removed: "Cflt: 2.2uF (eval) 1nF (datasheet) 16V 0603"
- note removed: "Rflt: 825R (eval), 100R (datasheet) 0.1% 0.1W 0603"
- moved on the sheet: C1, C2, C3, C4, C5, C7, C8, C9, D1, D2, JP5, L1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
